Commit message: add moveit pick&place demo

File: hdt_angler/hdt_angler_description/urdf/hdt_angler_a.xacro (robot description, xacro)
@@ -366,7 +366,7 @@
         </visual>
     </link>
-    <!-- endpoint -->
+    <!-- endpoint 0.17-->
     <joint name="endpoint_joint" type="fixed">
-        <origin xyz="0 0 0.17" rpy="${M_PI/2} ${-M_PI/2} 0"/>
+        <origin xyz="0 0 0.1" rpy="${M_PI/2} ${-M_PI/2} 0"/>
         <parent link="drive6_link"/>
         <child link="endpoint_link"/>
